File: KiCad Design/Baby Saving Project.kicad_sch (KiCad schematic)
At the start: 13 parts, among them Q1 BC107, U1 MPU-6050, U2 DHT11, U3 MAX30102, U4 ESP32-WROOM-32

Commit message: updated KiCad Design
Parts:
- removed BZ1: Buzzer, symbol Device:Buzzer
- removed Q1: BC107, Package_TO_SOT_THT:TO-18-3, symbol Transistor_BJT:BC107
- removed R2: 4.7k, symbol Device:R
- removed R3, R4, R6: 10k, symbol Device:R
- added D1, D2: LED, symbol Device:LED
- R1: value 4.7k -> 1k
Connections:
- net +3.3V: no longer R1.2
- net GND: now also D1.1 (K), D2.1 (K)
- net at U4.10 (IO25): no longer R5.1
- net at U4.24 (IO2): now also R5.1
- net at U4.29 (IO5): now also R1.1
- net at R5.2: now also D1.2 (A)
- new net: D2.2 (A), R1.2
